File: board/rpi-gpib-hat.kicad_pcb (KiCad board)
At the start: 2 copper layers, 65 x 30 mm, 6 parts, among them J1 RPI_GPIO, J2 GPIB

Commit message: Add project imprint and OSHW logo to board.
Parts:
- added OSHW: LOGO, local:OSHW, B.Cu at (127.4, 97.1)
Other:
- board text added: "Raspberry Pi GPIB µHat v0.1 github.com/Elemecca/rpi-gpib"
Changed lines of the file:
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@@
   (general
     (thickness 1.6)
-    (drawings 18)
+    (drawings 19)
     (tracks 0)
     (zones 0)
-    (modules 6)
+    (modules 7)
     (nets 49)
   )
@@
     (add_net GND)
   )
+  (module local:OSHW (layer B.Cu)
+    (at 127.382 97.108)
+    (descr "Imported from /home/sam/Downloads/oshw.svg")
+    (tags svg2mod)
+    (attr smd)
+    (fp_text reference OSHW (at 0 4.878245) (layer B.SilkS) hide
+      (effects (font (size 1.524 1.524) (thickness 0.3048)) (justify mirror))
+    )
+    (fp_text value LOGO (at 0 -4.878245) (layer B.SilkS) hide
+      (effects (font (size 1.524 1.524) (thickness 0.3048)) (justify mirror))
+    )
+    (fp_poly (pts (xy 2.009917 0.081788) (xy 1.510932 0.17458) (xy 1.481398 0.19998) (xy 1.328445 0.556819)
+      (xy 1.330872 0.595399) (xy 1.6216 1.019136) (xy 1.618414 1.053617) (xy 1.255293 1.416739)
+      (xy 1.220842 1.419928) (xy 0.789667 1.124038) (xy 0.750905 1.121215) (xy 0.404995 1.262815)
+      (xy 0.379496 1.292016) (xy 0.283426 1.808119) (xy 0.256807 1.830245) (xy -0.256778 1.830245)
+      (xy -0.283369 1.808119) (xy -0.379408 1.292016) (xy -0.404904 1.262815) (xy -0.750845 1.121215)
+      (xy -0.789607 1.124038) (xy -1.220751 1.419928) (xy -1.255233 1.416739) (xy -1.618385 1.053617)
+      (xy -1.621571 1.019136) (xy -1.330813 0.595399) (xy -1.328414 0.556819) (xy -1.481397 0.19998)
+      (xy -1.510931 0.17458) (xy -2.009886 0.081788) (xy -2.032015 0.055146) (xy -2.031984 -0.458408)
+      (xy -2.009855 -0.48505) (xy -1.523133 -0.575626) (xy -1.494236 -0.601224) (xy -1.342286 -0.980796)
+      (xy -1.34517 -1.019559) (xy -1.621632 -1.422442) (xy -1.618445 -1.456955) (xy -1.255263 -1.820077)
+      (xy -1.220781 -1.823266) (xy -0.82503 -1.551632) (xy -0.787087 -1.550221) (xy -0.612553 -1.643408)
+      (xy -0.583869 -1.632853) (xy -0.223996 -0.763309) (xy -0.234559 -0.7308) (xy -0.278238 -0.704046)
+      (xy -0.305859 -0.682879) (xy -0.443842 -0.558673) (xy -0.535025 -0.395419) (xy -0.567964 -0.204476)
+      (xy -0.539007 -0.024957) (xy -0.458375 0.130951) (xy -0.335428 0.253894) (xy -0.179521 0.33452)
+      (xy -0.000015 0.363474) (xy 0.179488 0.33452) (xy 0.335387 0.253894) (xy 0.458326 0.130951)
+      (xy 0.53895 -0.024957) (xy 0.567903 -0.204476) (xy 0.534972 -0.395419) (xy 0.443795 -0.558673)
+      (xy 0.305799 -0.682879) (xy 0.278237 -0.704046) (xy 0.234558 -0.7308) (xy 0.223994 -0.763309)
+      (xy 0.583838 -1.632884) (xy 0.612522 -1.643439) (xy 0.787056 -1.550255) (xy 0.824998 -1.551666)
+      (xy 1.22078 -1.823302) (xy 1.255232 -1.820113) (xy 1.618414 -1.456992) (xy 1.6216 -1.422479)
+      (xy 1.345108 -1.019593) (xy 1.342255 -0.980832) (xy 1.494205 -0.601257) (xy 1.523072 -0.57566)
+      (xy 2.009794 -0.485084) (xy 2.031923 -0.458442) (xy 2.031985 0.055107) (xy 2.009918 0.081777)
+      (xy 2.009917 0.081788)) (layer B.SilkS) (width 0.030354))
+  )
   (module lib:PinSocket_2x20_P2.54mm_Vertical_Centered_Anchor locked (layer F.Cu)
     (at 125.902 118.698 90)
@@
   (module local:NorComp_111-024-113L001 locked (layer B.Cu)
     (at 150.032 108.468)
-    (fp_text reference J2 (at 0.0508 6.8834) (layer B.SilkS)
+    (fp_text reference J2 (at 0.0508 6.8834 180 unlocked) (layer B.SilkS)
       (effects (font (size 1 1) (thickness 0.15)) (justify mirror))
     )
@@
       (net 3 GND))
   )
+  (gr_text "Raspberry Pi GPIB µHat v0.1\ngithub.com/Elemecca/rpi-gpib" (at 129.922 97.108 180) (layer B.SilkS)
+    (effects (font (size 1 1) (thickness 0.15)) (justify left mirror))
+  )
   (gr_text "Board Corner Radius = 3mm\nAll holes are M2.5" (at 184.278 127.334) (layer Cmts.User)

Commit message: Fix mounting holes to meet uHat spec.
Parts:
- H1, H2, H3, H4: footprint lib:MountingHole_2.7mm_M2.5_uHAT_RPi -> local:MountingHole_2.7mm_M2.5_uHAT
Changed lines of the file:
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@@
     (add_net GND)
   )
-  (module local:OSHW (layer B.Cu)
+  (module local:MountingHole_2.7mm_M2.5_uHAT locked (layer F.Cu)
+    (at 121.032 119.968)
+    (descr "Mounting Hole 2.7mm, no annular, M2.5")
+    (tags "mounting hole 2.7mm no annular m2.5")
+    (attr virtual)
+    (fp_text reference H1 (at 0 -3.7) (layer F.SilkS) hide
+      (effects (font (size 1 1) (thickness 0.15)))
+    )
+    (fp_text value MountingHole (at 0 3.7) (layer F.Fab) hide
+      (effects (font (size 1 1) (thickness 0.15)))
+    )
+    (fp_circle (center 0 0) (end 2.95 0) (layer F.CrtYd) (width 0.05))
+    (fp_text user %R (at 0.3 0) (layer F.Fab)
+      (effects (font (size 1 1) (thickness 0.15)))
+    )
+    (pad "" np_thru_hole circle (at 0 0) (size 2.7 2.7) (drill 2.7) (layers *.Cu *.Mask)
+      (solder_mask_margin 1.75) (clearance 1.75))
+  )
+  (module local:MountingHole_2.7mm_M2.5_uHAT locked (layer F.Cu)
+    (at 179.032 119.968)
+    (descr "Mounting Hole 2.7mm, no annular, M2.5")
+    (tags "mounting hole 2.7mm no annular m2.5")
+    (attr virtual)
+    (fp_text reference H2 (at 0 -3.7) (layer F.SilkS) hide
+      (effects (font (size 1 1) (thickness 0.15)))
+    )
+    (fp_text value MountingHole (at 0 3.7) (layer F.Fab) hide
+      (effects (font (size 1 1) (thickness 0.15)))
+    )
+    (fp_circle (center 0 0) (end 2.95 0) (layer F.CrtYd) (width 0.05))
+    (fp_text user %R (at 0.3 0) (layer F.Fab)
+      (effects (font (size 1 1) (thickness 0.15)))
+    )
+    (pad "" np_thru_hole circle (at 0 0) (size 2.7 2.7) (drill 2.7) (layers *.Cu *.Mask)
+      (solder_mask_margin 1.75) (clearance 1.75))
+  )
+  (module local:MountingHole_2.7mm_M2.5_uHAT locked (layer F.Cu)
+    (at 179.032 96.968)
+    (descr "Mounting Hole 2.7mm, no annular, M2.5")
+    (tags "mounting hole 2.7mm no annular m2.5")
+    (attr virtual)
+    (fp_text reference H3 (at 0 -3.7) (layer F.SilkS) hide
+      (effects (font (size 1 1) (thickness 0.15)))
+    )
+    (fp_text value MountingHole (at 0 3.7) (layer F.Fab) hide
+      (effects (font (size 1 1) (thickness 0.15)))
+    )
+    (fp_circle (center 0 0) (end 2.95 0) (layer F.CrtYd) (width 0.05))
+    (fp_text user %R (at 0.3 0) (layer F.Fab)
+      (effects (font (size 1 1) (thickness 0.15)))
+    )
+    (pad "" np_thru_hole circle (at 0 0) (size 2.7 2.7) (drill 2.7) (layers *.Cu *.Mask)
+      (solder_mask_margin 1.75) (clearance 1.75))
+  )
+  (module local:MountingHole_2.7mm_M2.5_uHAT locked (layer F.Cu)
+    (at 121.032 96.968)
+    (descr "Mounting Hole 2.7mm, no annular, M2.5")
+    (tags "mounting hole 2.7mm no annular m2.5")
+    (attr virtual)
+    (fp_text reference H4 (at 0 -3.7) (layer F.SilkS) hide
+      (effects (font (size 1 1) (thickness 0.15)))
+    )
+    (fp_text value MountingHole (at 0 3.7) (layer F.Fab) hide
+      (effects (font (size 1 1) (thickness 0.15)))
+    )
+    (fp_circle (center 0 0) (end 2.95 0) (layer F.CrtYd) (width 0.05))
+    (fp_text user %R (at 0.3 0) (layer F.Fab)
+      (effects (font (size 1 1) (thickness 0.15)))
+    )
+    (pad "" np_thru_hole circle (at 0 0) (size 2.7 2.7) (drill 2.7) (layers *.Cu *.Mask)
+      (solder_mask_margin 1.75) (clearance 1.75))
+  )
+  (module local:OSHW locked (layer B.Cu)
     (at 127.382 97.108)
     (descr "Imported from /home/sam/Downloads/oshw.svg")
@@
     )
   )
-  (module lib:MountingHole_2.7mm_M2.5_uHAT_RPi locked (layer F.Cu)
-    (at 121.032 119.968)
-    (descr "Mounting Hole 2.7mm, no annular, M2.5")
-    (tags "mounting hole 2.7mm no annular m2.5")
-    (attr virtual)
-    (fp_text reference H1 (at 0 -3.7) (layer F.SilkS) hide
-      (effects (font (size 1 1) (thickness 0.15)))
-    )
-    (fp_text value MountingHole (at 0 3.7) (layer F.Fab) hide
-      (effects (font (size 1 1) (thickness 0.15)))
-    )
-    (fp_text user %R (at 0.3 0) (layer F.Fab)
-      (effects (font (size 1 1) (thickness 0.15)))
-    )
-    (fp_circle (center 0 0) (end 2.7 0) (layer Cmts.User) (width 0.15))
-    (fp_circle (center 0 0) (end 2.95 0) (layer F.CrtYd) (width 0.05))
-    (pad "" np_thru_hole circle (at 0 0) (size 2.7 2.7) (drill 2.7) (layers *.Cu *.Mask)
-      (clearance 1.75))
-  )
-  (module lib:MountingHole_2.7mm_M2.5_uHAT_RPi locked (layer F.Cu)
-    (at 179.032 119.968)
-    (descr "Mounting Hole 2.7mm, no annular, M2.5")
-    (tags "mounting hole 2.7mm no annular m2.5")
-    (attr virtual)
-    (fp_text reference H2 (at 0 -3.7) (layer F.SilkS) hide
-      (effects (font (size 1 1) (thickness 0.15)))
-    )
-    (fp_text value MountingHole (at 0 3.7) (layer F.Fab) hide
-      (effects (font (size 1 1) (thickness 0.15)))
-    )
-    (fp_circle (center 0 0) (end 2.95 0) (layer F.CrtYd) (width 0.05))
-    (fp_circle (center 0 0) (end 2.7 0) (layer Cmts.User) (width 0.15))
-    (fp_text user %R (at 0.3 0) (layer F.Fab)
-      (effects (font (size 1 1) (thickness 0.15)))
-    )
-    (pad "" np_thru_hole circle (at 0 0) (size 2.7 2.7) (drill 2.7) (layers *.Cu *.Mask)
-      (clearance 1.75))
-  )
-  (module lib:MountingHole_2.7mm_M2.5_uHAT_RPi locked (layer F.Cu)
-    (at 179.032 96.968)
-    (descr "Mounting Hole 2.7mm, no annular, M2.5")
-    (tags "mounting hole 2.7mm no annular m2.5")
-    (attr virtual)
-    (fp_text reference H3 (at 0 -3.7) (layer F.SilkS) hide
-      (effects (font (size 1 1) (thickness 0.15)))
-    )
-    (fp_text value MountingHole (at 0 3.7) (layer F.Fab) hide
-      (effects (font (size 1 1) (thickness 0.15)))
-    )
-    (fp_text user %R (at 0.3 0) (layer F.Fab)
-      (effects (font (size 1 1) (thickness 0.15)))
-    )
-    (fp_circle (center 0 0) (end 2.7 0) (layer Cmts.User) (width 0.15))
-    (fp_circle (center 0 0) (end 2.95 0) (layer F.CrtYd) (width 0.05))
-    (pad "" np_thru_hole circle (at 0 0) (size 2.7 2.7) (drill 2.7) (layers *.Cu *.Mask)
-      (clearance 1.75))
-  )
-  (module lib:MountingHole_2.7mm_M2.5_uHAT_RPi locked (layer F.Cu)
-    (at 121.032 96.968)
-    (descr "Mounting Hole 2.7mm, no annular, M2.5")
-    (tags "mounting hole 2.7mm no annular m2.5")
-    (attr virtual)
-    (fp_text reference H4 (at 0 -3.7) (layer F.SilkS) hide
-      (effects (font (size 1 1) (thickness 0.15)))
-    )
-    (fp_text value MountingHole (at 0 3.7) (layer F.Fab) hide
-      (effects (font (size 1 1) (thickness 0.15)))
-    )
-    (fp_circle (center 0 0) (end 2.95 0) (layer F.CrtYd) (width 0.05))
-    (fp_circle (center 0 0) (end 2.7 0) (layer Cmts.User) (width 0.15))
-    (fp_text user %R (at 0.3 0) (layer F.Fab)
-      (effects (font (size 1 1) (thickness 0.15)))
-    )
-    (pad "" np_thru_hole circle (at 0 0) (size 2.7 2.7) (drill 2.7) (layers *.Cu *.Mask)
-      (clearance 1.75))
-  )
   (module local:NorComp_111-024-113L001 locked (layer B.Cu)

Commit message: Add courtyard for POE header.
Other:
- board text added: "POE"
Changed lines of the file:
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@@
   (general
     (thickness 1.6)
-    (drawings 19)
+    (drawings 24)
     (tracks 0)
     (zones 0)
@@
       (net 3 GND))
   )
+  (gr_text POE (at 179.032 113.828) (layer F.CrtYd)
+    (effects (font (size 1 1) (thickness 0.15)))
+  )
+  (gr_line (start 182.082 116.878) (end 182.082 110.778) (layer F.CrtYd) (width 0.05))
+  (gr_line (start 175.982 110.778) (end 175.982 116.878) (layer F.CrtYd) (width 0.05))
+  (gr_line (start 175.982 116.878) (end 182.082 116.878) (layer F.CrtYd) (width 0.05))
+  (gr_line (start 175.982 110.778) (end 182.082 110.778) (layer F.CrtYd) (width 0.05))
   (gr_text "Raspberry Pi GPIB µHat v0.1\ngithub.com/Elemecca/rpi-gpib" (at 129.922 97.108 180) (layer B.SilkS)
     (effects (font (size 1 1) (thickness 0.15)) (justify left mirror))
